Commit message: Adding IR macros with US macros

File: description/robot.urdf.xacro (robot description, xacro)
@@ -5,6 +5,7 @@
     <xacro:include filename="lidar.xacro"/>
     <!-- <xacro:include filename="camera.xacro"/> -->
-    <xacro:include filename="depth_camera.xacro"/>
+    <!-- <xacro:include filename="depth_camera.xacro"/> -->
     <xacro:include filename="imu.xacro"/>
     <xacro:include filename="ultrasonic.xacro"/>
+    <xacro:include filename="ir_sensor.xacro"/>
 </robot>

File: description/ultrasonic.xacro (robot description, xacro)
@@ -1,10 +1,10 @@
 <?xml version="1.0"?>
 <robot xmlns:xacro="http://www.ros.org/wiki/xacro">
-    <joint name="ir_sensor_joint" type="fixed">
-        <origin xyz="0.305 0.2 0.016" rpy="0 0 0"/>
+    <joint name="ultrasonic_1_joint" type="fixed">
+        <origin xyz="0.305 0.05 0.5 " rpy="0 0 0"/>
         <parent link="chassis"/>
-        <child link="ir_sensor_link"/>
+        <child link="ultrasonic_1_link"/>
     </joint>
-    <link name="ir_sensor_link">
+    <link name="ultrasonic_1_link">
         <collision>
             <origin xyz="0 0 0" rpy="0 0 0"/>
@@ -18,5 +18,5 @@
                 <box size="0.02 0.02 0.02"/>
             </geometry>
-             <material>Gazebo/Green</material>
+            <material name="iRobot/Green"/>
         </visual>
         <inertial>
@@ -26,56 +26,42 @@
         </inertial>
     </link>
-    <!-- <gazebo reference="imu_sensor_link">
-        <gravity>true</gravity>
-        <sensor name='imu_sensor' type='imu'>
-            <always_on>1</always_on>
-            <update_rate>1000</update_rate>
-            <visualize>1</visualize>
-            <topic>imu_topic</topic>
-            <plugin name='imu' filename='libgazebo_ros_imu_sensor.so'>
-                <topicName>imu_data</topicName>
-                <bodyName>imu_sensor_link</bodyName>
-                <updateRateHZ>10.0</updateRateHZ>
-                <gaussianNoise>0.0</gaussianNoise>
-                <xyzOffset>0 0 0</xyzOffset>
-                <rpyOffset>0 0 0</rpyOffset>
-            </plugin>
-            <pose>0 0 0 0 0 0</pose>
-        </sensor>
-    </gazebo> -->
-    <gazebo reference="ir_sensor_link">
-        <sensor type="ray" name="TeraRanger">
+    <gazebo reference="ultrasonic_1_link">
+        <sensor type="ray" name="ultrasonics_1">
             <pose>0 0 0 0 0 0</pose>
             <visualize>true</visualize>
-            <update_rate>50</update_rate>
+            <update_rate>5</update_rate>
             <ray>
                 <scan>
                     <horizontal>
-                    <samples>10</samples>
-                    <resolution>1</resolution>
-                    <min_angle>-0.14835</min_angle>
-                    <max_angle>0.14835</max_angle>
+                    <samples>5</samples>
+                    <resolution>1.000000</resolution>
+                    <min_angle>-0.12</min_angle>
+                    <max_angle>0.12</max_angle>
                     </horizontal>
                     <vertical>
                     <samples>10</samples>
-                    <resolution>1</resolution>
-                    <min_angle>-0.14835</min_angle>
-                    <max_angle>0.14835</max_angle>
+                    <resolution>1.000000</resolution>
+                    <min_angle>-0.1</min_angle>
+                    <max_angle>0.1</max_angle>
                     </vertical>
                 </scan>
                 <range>
-                    <min>0.01</min>
-                    <max>2</max>
-                    <resolution>0.02</resolution>
+                    <min>0.02</min>
+                    <max>4</max>
+                    <resolution>0.001</resolution>
                 </range>
+                <noise>
+                    <type>gaussian</type>
+                    <mean>0.0</mean>
+                    <stddev>0.01</stddev>
+                </noise>
             </ray>
-            <plugin filename="libgazebo_ros_range.so" name="gazebo_ros_range">
-                <gaussianNoise>0.005</gaussianNoise>
-                <alwaysOn>true</alwaysOn>
-                <updateRate>50</updateRate>
-                <topicName>sensor/ir_front</topicName>
-                <frameName>base_ir_front</frameName>
-                <radiation>INFRARED</radiation>
-                <fov>0.2967</fov>
+            <plugin name="ultrasonic_sensor_1" filename="libgazebo_ros_ray_sensor.so">
+                <ros>
+                    <remapping>~/out:=ultrasonic_sensor_1</remapping>
+                </ros>
+                <output_type>sensor_msgs/Range</output_type>
+                <radiation_type>ultrasound</radiation_type>
+                <frame_name>ultrasonic_1_link</frame_name>
             </plugin>
         </sensor>
