Commit message: adding rviz in the launch file

File: description/lidar.xacro (robot description, xacro)
@@ -26,5 +26,5 @@
         <sensor name="laser" type="ray">
             <pose>0 0 0 0 0 0</pose>
-            <visualize>false</visualize>
+            <visualize>true</visualize>
             <updateRate>10</updateRate>
             <ray>

File: description/robot_core.xacro (robot description, xacro)
@@ -17,4 +17,7 @@
         <color rgba="1 0 0 1"/>
     </material>
+    <material name="Cyan">
+        <color rgba="0 1.0 1.0 1.0"/>
+      </material>
     <!-- BASE LINK  -->
     <link name="base_link">
@@ -32,5 +35,5 @@
                 <box size="0.3 0.3 0.15"/>
             </geometry>
-            <material name="white"/>
+            <material name="Cyan"/>
         </visual>
         <collision>
